Commit message: Modify URDF to include table, ee

File: lbr_description/gazebo/lbr_gazebo.xacro (robot description, xacro)
@@ -38,4 +38,12 @@
         <xacro:gazebo_joint_reference name="A7" />
         <xacro:gazebo_link_reference name="link_7" />
+        <xacro:gazebo_joint_reference name="joint_ee" />
+        <xacro:gazebo_link_reference name="link_ee" />
+        <xacro:gazebo_joint_reference name="joint_drillbit" />
+        <xacro:gazebo_link_reference name="link_drillbit" />
+        <xacro:gazebo_joint_reference name="joint_tool" />
+        <xacro:gazebo_link_reference name="link_tool" />
+        <xacro:gazebo_joint_reference name="world_plank_joint" />
+        <xacro:gazebo_link_reference name="plank" />
     </xacro:macro>
 </robot>

File: lbr_description/urdf/med7/med7.urdf.xacro (robot description, xacro)
@@ -15,4 +15,8 @@
         <child link="link_0" />
     </joint>
+    <joint name="world_plank_joint" type="fixed">
+        <parent link="world" />
+        <child link="plank" />
+    </joint>
     <!-- med -->
     <xacro:med7 robot_name="$(arg robot_name)" port_id="$(arg port_id)" sim="$(arg sim)" />

File: lbr_description/urdf/med7/med7_description.urdf.xacro (robot description, xacro)
@@ -21,9 +21,33 @@
     <xacro:property name="effort_limit" value="200" />
     <!-- includes -->
-    <xacro:include filename="$(find lbr_description)/gazebo/lbr.gazebo.xacro" />
+    <xacro:include filename="$(find lbr_description)/gazebo/lbr_gazebo.xacro" />
     <xacro:include filename="$(find lbr_ros2_control)/config/lbr_system_interface.xacro" />
     <!-- robot as extracted via https://github.com/syuntoku14/fusion2urdf -->
     <xacro:macro name="med7"
         params="robot_name:=^|lbr port_id:=^|30200 sim:=^|true">
+        <link name="plank">
+            <inertial>
+                <origin rpy="0 0 0" xyz="-0.001896 0.0 0.076263" />
+                <mass value="7.143112" />
+                <inertia ixx="0.038694" ixy="0.0" ixz="-0.000686" iyy="0.039461" iyz="0.0"
+                    izz="0.054387" />
+            </inertial>
+            <visual>
+                <origin rpy="0 0 0" xyz="-0.47 0 -0.017" />
+                <geometry>
+                    <box size="0.64 1.1 0.02"/>
+                </geometry>
+                <material name="gray">
+                    <color rgba="0.5 0.5 0.5 1.0" />
+                </material>
+            </visual>
+            <!-- maybe need to turn this on, for now it is off for spawning in gazebo -->
+            <!-- <collision>
+                <origin rpy="0 0 0" xyz="-0.47 0 -0.017" />
+                <geometry>
+                    <box size="0.64 1.1 0.02"/>
+                </geometry>
+            </collision> -->
+        </link>
         <link name="link_0">
             <inertial>
@@ -266,23 +290,64 @@
                 <inertia ixx="0.008179" ixy="0.0" ixz="0.0" iyy="0.006879" iyz="0.002704" izz="0.003709" />
             </inertial>
-            <visual>
+            <!-- <visual>
+                <origin rpy="0 0 0" xyz="-0.066 -0.033 0" />
+                <geometry>
+                    <mesh filename="package://lbr_description/meshes/med7/visual/finalshiftedee.STL" scale="0.001 0.001 0.001" />
+                </geometry>
+                <material name="gray">
+                    <color rgba="0.5 0.5 0.5 1.0" />
+                </material>
+            </visual> -->
+            <visual>
+                <origin rpy="0 0 3.1415926" xyz="0 0 0" />
+                <geometry>
+                    <mesh filename="package://lbr_description/meshes/med7/visual/finalshiftedee.STL" scale="0.001 0.001 0.001" />
+                </geometry>
+                <material name="gray">
+                    <color rgba="0.5 0.5 0.5 1.0" />
+                </material>
+            </visual>
+            <collision>
                 <origin rpy="0 0 0" xyz="0.0 0.0 0.10" />
                 <geometry>
-                    <cylinder length="0.2" radius="0.02" />
-                </geometry>
-            </visual>
-            <collision>
-                <origin rpy="0 0 0" xyz="0.0 0.0 0.10" />
-                <geometry>
-                    <cylinder length="0.2" radius="0.02" />
+                    <cylinder length="0.218" radius="0.04" />
+                </geometry>
+            </collision>
+        </link>
+        <!-- change the values because ee is not cylinder of 20,2 cm -->
+        <joint name="joint_drillbit" type="fixed">
+            <parent link="link_ee" />
+            <child link="link_drillbit" />
+            <origin xyz="0 0 0.2" rpy="0 0 0" />
+        </joint>
+        <link name="link_drillbit">
+            <inertial>
+                <origin rpy="0 0 0" xyz="0.0 -0.029824 0.076267" />
+                <mass value="1.474048" />
+                <inertia ixx="0.008179" ixy="0.0" ixz="0.0" iyy="0.006879" iyz="0.002704" izz="0.003709" />
+            </inertial>
+            <visual>
+                <origin rpy="0 0 0" xyz="0.0 0.0 0.0375" />
+                <geometry>
+                    <cylinder length="0.0326" radius="0.0028" />
+                </geometry>
+                <material name="gray">
+                    <color rgba="0.5 0.5 0.5 1.0" />
+                </material>
+            </visual>
+            <collision>
+                <origin rpy="0 0 0" xyz="0.0 0.0 0.0375" />
+                <geometry>
+                    <cylinder length="0.0326" radius="0.0028" />
                 </geometry>
             </collision>
         </link>
         <joint name="joint_tool" type="fixed">
-            <parent link="link_ee" />
+            <parent link="link_drillbit" />
             <child link="link_tool" />
-            <origin xyz="0 0 0.2" rpy="0 0 0" />
+            <origin xyz="0 0 0.0326" rpy="0 0 0" />
         </joint>
         <link name="link_tool">
+        <!-- tip stub -->
         </link>
         <xacro:lbr_gazebo robot_name="${robot_name}" />
